File: eFuse.sch (KiCad schematic (older format))
At the start: 8 parts, among them U3 TPS25921x

Commit message: Added product info and Schematic
Parts:
- removed U3: TPS25921x, LMS-6_Interface_Board:SOIC-8_W5.4mm, symbol power_LMS6:TPS25921x
- added U3: TPS25921ADR, LMS-6_Interface_Board:SOIC-8_W5.4mm, symbol power_LMS6:TPS25921ADR
Connections:
- net GND: now also U3.1 (GND)
- net eFuse_In: now also U3.4 (IN)
- net eFuse_Out: now also U3.5 (OUT)
- net at C10.1: now also U3.2 (SS)
- net at R6.2, R7.1: now also U3.3 (ENUV)
- net at R9.1: now also U3.6 (~FLT~)
- net at R10.1: now also U3.7 (ILIM)
- net at R7.2, R8.1: now also U3.8 (OVP)
Changed lines of the file:
@@
 $EndDescr
-$Comp
-L power_LMS6:TPS25921x U3
-U 1 1 5F9193A1
-P 5600 3050
-F 0 "U3" H 5550 4015 50  0000 C CNN
-F 1 "TPS25921x" H 5550 3924 50  0000 C CNN
-F 2 "LMS-6_Interface_Board:SOIC-8_W5.4mm" H 5530 3890 50  0001 C CNN
-F 3 "https://www.ti.com/lit/ds/symlink/tps25921l.pdf" H 5530 3890 50  0001 C CNN
-	1    5600 3050
-	1    0    0    -1
-$EndComp
 $Comp
 L Device:R_US R?
@@
 Text Notes 7450 2300 0    50   ~ 0
 Power Failure Detection Threshold: ... 4.62V\nRelease UVLO, Enable Chip: ............... 4.79V\nOver Voltage Cut-off: ....................... 16.76V\nRelease OV: ..................................... 16.16 V\n\nCurrent LImit: ..................................  1.51 A\nCurrent LImit Fast Trip: .................... 2.39 A
+$Comp
+L power_LMS6:TPS25921ADR U3
+U 1 1 5F934945
+P 5600 3050
+F 0 "U3" H 5550 4015 50  0000 C CNN
+F 1 "TPS25921ADR" H 5550 3924 50  0000 C CNN
+F 2 "LMS-6_Interface_Board:SOIC-8_W5.4mm" H 5530 3890 50  0001 C CNN
+F 3 "https://www.ti.com/lit/ds/symlink/tps25921l.pdf" H 5530 3890 50  0001 C CNN
+F 4 "Texas Instruments" H 5550 4015 50  0001 C CNN "Manufacturer"
+F 5 "TPS25921ADR" H 5550 3924 50  0001 C CNN "MPN"
+	1    5600 3050
+	1    0    0    -1
+$EndComp
 $EndSCHEMATC

Commit message: Rev C Board layout
Parts:
- D1: footprint digikey-footprints:0805 -> LED_SMD:LED_0805_2012Metric_Pad1.15x1.40mm_HandSolder
Changed lines of the file:
@@
 $Descr USLetter 11000 8500
 encoding utf-8
-Sheet 5 5
+Sheet 5 6
 Title "eFuse"
 Date "2020-10-17"
@@
 F 0 "D1" H 5000 2237 60  0000 C CNN
 F 1 "LH_R974-LP-1" H 5000 2131 60  0000 C CNN
-F 2 "digikey-footprints:0805" H 5250 2100 60  0001 L CNN
+F 2 "LED_SMD:LED_0805_2012Metric_Pad1.15x1.40mm_HandSolder" H 5250 2100 60  0001 L CNN
 F 3 "https://dammedia.osram.info/media/resource/hires/osram-dam-2493888/LH%20R974.pdf" H 5250 2200 60  0001 L CNN
 F 4 "475-1415-1-ND" H 5250 2300 60  0001 L CNN "Digi-Key_PN"
