File: CardEdgeConn.sch (KiCad schematic (older format))
At the start: 8 parts, among them J13 Conn_01x02, J5 5-5530843-4, J6 Conn_01x03, J7 302-S101

Commit message: Changed J9 connections to help with layout.
Parts:
- J5: footprint (none) -> Connector_PinHeader_2.54mm:PinHeader_2x20_P2.54mm_Vertical
- JP1, JP2: footprint SMT-JUMPER_3_1-NC -> Jumpers:SMT-JUMPER_3_1-NC_TRACE_NO-SILK
Changed lines of the file:
@@
 F 0 "J5" H 3150 5425 50  0000 C CNN
 F 1 "5-5530843-4" H 3150 5334 50  0000 C CNN
-F 2 "" H 3150 3200 50  0001 C CNN
+F 2 "Connector_PinHeader_2.54mm:PinHeader_2x20_P2.54mm_Vertical" H 3150 3200 50  0001 C CNN
 F 3 "https://www.te.com/commerce/DocumentDelivery/DDEController?Action=srchrtrv&DocNm=5530843&DocType=Customer+Drawing&DocLang=English" H 3150 3200 50  0001 C CNN
 F 4 "5-5530843-4" H 3150 3200 50  0001 C CNN "MPN"
@@
 U 1 1 5F8B7A4C
 P 1300 3700
-F 0 "JP1" H 1404 3795 45  0000 L CNN
-F 1 "JUMPER-SMT_3_1-NC" H 1404 3711 45  0000 L CNN
-F 2 "SMT-JUMPER_3_1-NC" H 1300 3950 20  0001 C CNN
+F 0 "JP1" H 1404 3605 45  0000 L CNN
+F 1 "JUMPER-SMT_3_1-NC" H 1404 3689 45  0000 L CNN
+F 2 "Jumpers:SMT-JUMPER_3_1-NC_TRACE_NO-SILK" H 1300 3950 20  0001 C CNN
 F 3 "" V 1300 3645 60  0001 C CNN
-F 4 "XXX-00000" H 1404 3616 60  0000 L CNN "PROD_ID"
+F 4 "XXX-00000" H 1404 3784 60  0000 L CNN "PROD_ID"
 	1    1300 3700
 	1    0    0    1
@@
 F 0 "JP2" H 5454 3605 45  0000 L CNN
 F 1 "JUMPER-SMT_3_1-NC" H 5454 3689 45  0000 L CNN
-F 2 "SMT-JUMPER_3_1-NC" H 5350 3950 20  0001 C CNN
+F 2 "Jumpers:SMT-JUMPER_3_1-NC_TRACE_NO-SILK" H 5350 3950 20  0001 C CNN
 F 3 "" V 5350 3645 60  0001 C CNN
 F 4 "XXX-00000" H 5454 3784 60  0000 L CNN "PROD_ID"

Commit message: Fixed DRC Errors
Fixed drc errors
Parts:
- removed J7: 302-S101, digikey-footprints:PinHeader_2x5_P2.54mm_Drill1.2mm, symbol Connector_Generic:Conn_02x05_Odd_Even
Changed lines of the file:
@@
 Title "Card Connector"
 Date "2020-10-17"
-Rev "6"
+Rev "7"
 Comp ""
 Comment1 ""
@@
 Text HLabel 2250 1300 0    50   Input ~ 0
 ST7-ICCCLK
-$Comp
-L Connector_Generic:Conn_02x05_Odd_Even J7
-U 1 1 5F836EA0
-P 8300 2650
-F 0 "J7" H 8350 3067 50  0000 C CNN
-F 1 "302-S101" H 8350 2976 50  0000 C CNN
-F 2 "digikey-footprints:PinHeader_2x5_P2.54mm_Drill1.2mm" H 8300 2650 50  0001 C CNN
-F 3 "http://www.on-shore.com/wp-content/uploads/2018/04/302-SXX1.pdf" H 8300 2650 50  0001 C CNN
-F 4 "302-S101" H 8300 2650 50  0001 C CNN "MPN"
-F 5 "On Shore Technology Inc." H 8300 2650 50  0001 C CNN "Maufacturer"
-	1    8300 2650
-	1    0    0    -1
-$EndComp
-Text HLabel 8600 2750 2    50   Input ~ 0
-ST7-ICCSEL
-Text HLabel 8600 2450 2    50   Input ~ 0
-ST7-ICCDATA
-Text HLabel 8600 2650 2    50   Input ~ 0
-ST7-RESET
-Text HLabel 8600 2550 2    50   Input ~ 0
-ST7-ICCCLK
-$Comp
-L power:VDD #PWR?
-U 1 1 5F83EE0B
-P 7550 2650
-AR Path="/5F83EE0B" Ref="#PWR?"  Part="1"
-AR Path="/5F7BE189/5F83EE0B" Ref="#PWR?"  Part="1"
-AR Path="/5F7C6408/5F83EE0B" Ref="#PWR015"  Part="1"
-F 0 "#PWR015" H 7550 2500 50  0001 C CNN
-F 1 "VDD" H 7565 2823 50  0000 C CNN
-F 2 "" H 7550 2650 50  0001 C CNN
-F 3 "" H 7550 2650 50  0001 C CNN
-	1    7550 2650
-	1    0    0    -1
-$EndComp
-Wire Wire Line
-	8100 2750 7550 2750
-Wire Wire Line
-	7550 2750 7550 2650
-$Comp
-L power:GND #PWR?
-U 1 1 5F840CF8
-P 8000 3000
-AR Path="/5F840CF8" Ref="#PWR?"  Part="1"
-AR Path="/5F7BE189/5F840CF8" Ref="#PWR?"  Part="1"
-AR Path="/5F7C6408/5F840CF8" Ref="#PWR016"  Part="1"
-F 0 "#PWR016" H 8000 2750 50  0001 C CNN
-F 1 "GND" H 8005 2827 50  0000 C CNN
-F 2 "" H 8000 3000 50  0001 C CNN
-F 3 "" H 8000 3000 50  0001 C CNN
-	1    8000 3000
-	1    0    0    -1
-$EndComp
-Wire Wire Line
-	8000 2450 8100 2450
-Wire Wire Line
-	8000 2450 8000 2550
-Wire Wire Line
-	8100 2650 8000 2650
-Connection ~ 8000 2650
-Wire Wire Line
-	8000 2650 8000 3000
-Wire Wire Line
-	8100 2550 8000 2550
-Connection ~ 8000 2550
-Wire Wire Line
-	8000 2550 8000 2650
-$Comp
-L power:GND #PWR?
-U 1 1 5F845227
-P 8650 3000
-AR Path="/5F845227" Ref="#PWR?"  Part="1"
-AR Path="/5F7BE189/5F845227" Ref="#PWR?"  Part="1"
-AR Path="/5F7C6408/5F845227" Ref="#PWR017"  Part="1"
-F 0 "#PWR017" H 8650 2750 50  0001 C CNN
-F 1 "GND" H 8655 2827 50  0000 C CNN
-F 2 "" H 8650 3000 50  0001 C CNN
-F 3 "" H 8650 3000 50  0001 C CNN
-	1    8650 3000
-	1    0    0    -1
-$EndComp
-Wire Wire Line
-	8600 2850 8650 2850
-Wire Wire Line
-	8650 2850 8650 3000
 Text HLabel 4350 1800 2    50   Input ~ 0
 HEADER1.1
@@
 L power:+9V #PWR?
 U 1 1 5F8BD332
-P 4050 4500
+P 4350 4500
 AR Path="/5F8BD332" Ref="#PWR?"  Part="1"
 AR Path="/5F7BE189/5F8BD332" Ref="#PWR?"  Part="1"
 AR Path="/5F7C6408/5F8BD332" Ref="#PWR014"  Part="1"
-F 0 "#PWR014" H 4050 4350 50  0001 C CNN
-F 1 "+9V" H 4065 4673 50  0000 C CNN
-F 2 "" H 4050 4500 50  0001 C CNN
-F 3 "" H 4050 4500 50  0001 C CNN
-	1    4050 4500
-	1    0    0    -1
-$EndComp
-Wire Wire Line
-	4050 4700 4050 4500
+F 0 "#PWR014" H 4350 4350 50  0001 C CNN
+F 1 "+9V" H 4365 4673 50  0000 C CNN
+F 2 "" H 4350 4500 50  0001 C CNN
+F 3 "" H 4350 4500 50  0001 C CNN
+	1    4350 4500
+	1    0    0    -1
+$EndComp
+Wire Wire Line
+	4350 4700 4350 4500
 $Comp
 L power:+BATT #PWR?
@@
 	1    0    0    -1
 $EndComp
-Wire Wire Line
-	3550 4700 4050 4700
 Wire Wire Line
 	3750 4500 3750 4600
@@
 	-1   0    0    -1
 $EndComp
+$Comp
+L power:PWR_FLAG #FLG0104
+U 1 1 5F9F7887
+P 2500 1200
+F 0 "#FLG0104" H 2500 1275 50  0001 C CNN
+F 1 "PWR_FLAG" V 2500 1327 50  0000 L CNN
+F 2 "" H 2500 1200 50  0001 C CNN
+F 3 "~" H 2500 1200 50  0001 C CNN
+	1    2500 1200
+	0    -1   -1   0
+$EndComp
+$Comp
+L power:PWR_FLAG #FLG0105
+U 1 1 5F9F87AF
+P 1700 3100
+F 0 "#FLG0105" H 1700 3175 50  0001 C CNN
+F 1 "PWR_FLAG" H 1700 3273 50  0000 C CNN
+F 2 "" H 1700 3100 50  0001 C CNN
+F 3 "~" H 1700 3100 50  0001 C CNN
+	1    1700 3100
+	-1   0    0    1
+$EndComp
+Connection ~ 1700 3100
+$Comp
+L power:PWR_FLAG #FLG0106
+U 1 1 5F9F8AAB
+P 3750 4600
+F 0 "#FLG0106" H 3750 4675 50  0001 C CNN
+F 1 "PWR_FLAG" V 3750 4728 50  0000 L CNN
+F 2 "" H 3750 4600 50  0001 C CNN
+F 3 "~" H 3750 4600 50  0001 C CNN
+	1    3750 4600
+	0    1    1    0
+$EndComp
+Connection ~ 3750 4600
+Wire Wire Line
+	3550 4700 4350 4700
 $EndSCHEMATC

Commit message: Final updates to REV B
Parts:
- removed J5: 5-5530843-4, Connector_PinHeader_2.54mm:PinHeader_2x20_P2.54mm_Vertical, symbol Programmer_Board:5-5530843-4
- added J5: EBC20DRAS, LMS-6_Interface_Board:EBC20DRAS, symbol LMS-6_Interface_Connector:EBC20DRAS
Connections:
- net +9V: now also J5.39 (Pin_39), J5.40 (Pin_40)
- net +BATT: now also J5.31 (Pin_31)
- net GND: now also J5.10 (Pin_10), J5.15 (Pin_15), J5.16 (Pin_16), J5.19 (Pin_19), J5.20 (Pin_20), J5.33 (Pin_33), J5.34 (Pin_34), J5.9 (Pin_9)
- net HEADER1.1: now also J5.14 (Pin_14)
- net HEADER1.10: now also J5.37 (Pin_37)
- net HEADER1.2: now also J5.22 (Pin_22)
- net HEADER1.3: now also J5.24 (Pin_24)
- net HEADER1.4: now also J5.28 (Pin_28)
- net HEADER1.5: now also J5.25 (Pin_25)
- net HEADER1.6: now also J5.27 (Pin_27)
- net HEADER1.7: now also J5.29 (Pin_29)
- net HEADER1.9: now also J5.35 (Pin_35)
- net J5.2: now also J5.11 (Pin_11)
- net J5.3: now also J5.32 (Pin_32)
- net ST7-ICCCLK: now also J5.3 (Pin_3)
- net ST7-ICCDATA: now also J5.6 (Pin_6)
- net ST7-ICCSEL: now also J5.4 (Pin_4)
- net ST7-RESET: now also J5.5 (Pin_5)
- net SW1.1: now also J5.18 (Pin_18)
- net SW1.2: now also J5.17 (Pin_17)
- net SW1.3: now also J5.36 (Pin_36)
- net SW1.4: now also J5.13 (Pin_13)
- net U21.20-DCLK: now also J5.12 (Pin_12)
- net U22.3: now also J5.30 (Pin_30)
- net U3.18: now also J5.38 (Pin_38)
- net U3.19: now also J5.21 (Pin_21)
- net VDD: now also J5.1 (Pin_1), J5.2 (Pin_2), J5.7 (Pin_7), J5.8 (Pin_8)
- net at JP1.3, JP2.1: now also J5.23 (Pin_23)
- net at JP1.1, JP2.3: now also J5.26 (Pin_26)
Changed lines of the file:
@@
 Title "Card Connector"
 Date "2020-10-17"
-Rev "7"
+Rev "9"
 Comp ""
 Comment1 ""
@@
 F 3 "" H 3650 3250 50  0001 C CNN
 	1    3650 3250
-	1    0    0    -1
-$EndComp
-$Comp
-L Programmer_Board:5-5530843-4 J?
-U 1 1 5F7D09C4
-P 3150 3200
-AR Path="/5F7D09C4" Ref="J?"  Part="1"
-AR Path="/5F7BE189/5F7D09C4" Ref="J?"  Part="1"
-AR Path="/5F7C6408/5F7D09C4" Ref="J5"  Part="1"
-F 0 "J5" H 3150 5425 50  0000 C CNN
-F 1 "5-5530843-4" H 3150 5334 50  0000 C CNN
-F 2 "Connector_PinHeader_2.54mm:PinHeader_2x20_P2.54mm_Vertical" H 3150 3200 50  0001 C CNN
-F 3 "https://www.te.com/commerce/DocumentDelivery/DDEController?Action=srchrtrv&DocNm=5530843&DocType=Customer+Drawing&DocLang=English" H 3150 3200 50  0001 C CNN
-F 4 "5-5530843-4" H 3150 3200 50  0001 C CNN "MPN"
-F 5 "TE Connectivity AMP Connectors" H 3150 3200 50  0001 C CNN "Manufacturer"
-	1    3150 3200
 	1    0    0    -1
 $EndComp
@@
 Wire Wire Line
 	3550 4700 4350 4700
+$Comp
+L LMS-6_Interface_Connector:EBC20DRAS J5
+U 1 1 5F8E17E9
+P 3100 2100
+F 0 "J5" H 3150 3217 50  0000 C CNN
+F 1 "EBC20DRAS" H 3150 3126 50  0000 C CNN
+F 2 "LMS-6_Interface_Board:EBC20DRAS" H 3100 2100 50  0001 C CNN
+F 3 "https://drawings-pdf.s3.amazonaws.com/C10876.pdf" H 3100 2100 50  0001 C CNN
+	1    3100 2100
+	1    0    0    -1
+$EndComp
 $EndSCHEMATC

Commit message: Rev C Board layout
Parts:
- D3: footprint digikey-footprints:0805 -> LED_SMD:LED_0805_2012Metric_Pad1.15x1.40mm_HandSolder
Changed lines of the file:
@@
 $Descr USLetter 11000 8500
 encoding utf-8
-Sheet 4 5
+Sheet 5 5
 Title "Card Connector"
 Date "2020-10-17"
@@
 	3400 1800 4350 1800
 $Comp
-L power:+9V #PWR?
-U 1 1 5F8BD332
-P 4350 4500
-AR Path="/5F8BD332" Ref="#PWR?"  Part="1"
-AR Path="/5F7BE189/5F8BD332" Ref="#PWR?"  Part="1"
-AR Path="/5F7C6408/5F8BD332" Ref="#PWR014"  Part="1"
-F 0 "#PWR014" H 4350 4350 50  0001 C CNN
-F 1 "+9V" H 4365 4673 50  0000 C CNN
-F 2 "" H 4350 4500 50  0001 C CNN
-F 3 "" H 4350 4500 50  0001 C CNN
-	1    4350 4500
-	1    0    0    -1
-$EndComp
-Wire Wire Line
-	4350 4700 4350 4500
-$Comp
 L power:+BATT #PWR?
 U 1 1 5F8C0163
@@
 F 0 "D3" H 6450 4237 60  0000 C CNN
 F 1 "LG R971-KN-1" H 6450 4131 60  0000 C CNN
-F 2 "digikey-footprints:0805" H 6700 4100 60  0001 L CNN
+F 2 "LED_SMD:LED_0805_2012Metric_Pad1.15x1.40mm_HandSolder" H 6700 4100 60  0001 L CNN
 F 3 "https://dammedia.osram.info/media/resource/hires/osram-dam-2493888/LH%20R974.pdf" H 6700 4200 60  0001 L CNN
 F 4 "475-1410-1-ND" H 6700 4300 60  0001 L CNN "Digi-Key_PN"
@@
 $EndComp
 Connection ~ 3750 4600
-Wire Wire Line
-	3550 4700 4350 4700
 $Comp
 L LMS-6_Interface_Connector:EBC20DRAS J5
@@
 	1    0    0    -1
 $EndComp
+$Comp
+L power:+9V #PWR?
+U 1 1 5F8BD332
+P 4350 4500
+AR Path="/5F8BD332" Ref="#PWR?"  Part="1"
+AR Path="/5F7BE189/5F8BD332" Ref="#PWR?"  Part="1"
+AR Path="/5F7C6408/5F8BD332" Ref="#PWR014"  Part="1"
+F 0 "#PWR014" H 4350 4350 50  0001 C CNN
+F 1 "+9V" H 4365 4673 50  0000 C CNN
+F 2 "" H 4350 4500 50  0001 C CNN
+F 3 "" H 4350 4500 50  0001 C CNN
+	1    4350 4500
+	1    0    0    -1
+$EndComp
+Wire Wire Line
+	3550 4700 4350 4700
+Wire Wire Line
+	4350 4700 4350 4500
 $EndSCHEMATC
