File: DC-DC Converter.sch (KiCad schematic (older format))
At the start: 4 parts, among them U2 TEC2-1219WI

Commit message: Fixed DRC Errors
Fixed drc errors
Changed lines of the file:
@@
 Title "DC-DC Converter"
 Date "2020-10-17"
-Rev "6"
+Rev "7"
 Comp ""
 Comment1 ""
@@
 	7850 4150 7850 4400
 Wire Wire Line
-	6000 3750 6800 3750
+	6000 3750 6500 3750
 Wire Wire Line
 	6000 4050 6000 4150
@@
 Wire Wire Line
 	6750 3950 6800 3950
+$Comp
+L power:PWR_FLAG #FLG0103
+U 1 1 5F9D90BB
+P 6500 3750
+F 0 "#FLG0103" H 6500 3825 50  0001 C CNN
+F 1 "PWR_FLAG" H 6500 3923 50  0000 C CNN
+F 2 "" H 6500 3750 50  0001 C CNN
+F 3 "~" H 6500 3750 50  0001 C CNN
+	1    6500 3750
+	1    0    0    -1
+$EndComp
+Connection ~ 6500 3750
+Wire Wire Line
+	6500 3750 6800 3750
 $EndSCHEMATC

Commit message: Fixing component field names, because I can't spell.
Parts:
- L1: MPN (none) -> TCK-154; Manufacturer (none) -> Traco Power; Manufacturer_Name Traco Power -> (none); Manufacturer_Part_Number TCK-154 -> (none)
Changed lines of the file:
@@
 F 6 "495-TCK-154" H 5800 3400 50  0001 L CNN "Mouser Part Number"
 F 7 "https://www.mouser.co.uk/ProductDetail/TRACO-Power/TCK-154?qs=w%2Fv1CP2dgqrcxTwKbnHwhQ%3D%3D" H 5800 3300 50  0001 L CNN "Mouser Price/Stock"
-F 8 "Traco Power" H 5800 3200 50  0001 L CNN "Manufacturer_Name"
-F 9 "TCK-154" H 5800 3100 50  0001 L CNN "Manufacturer_Part_Number"
+F 8 "Traco Power" H 5800 3200 50  0001 L CNN "Manufacturer"
+F 9 "TCK-154" H 5800 3100 50  0001 L CNN "MPN"
 	1    5150 3750
 	1    0    0    -1

Commit message: Added product info and Schematic
Parts:
- C9: MPN C3216X7R1E475K160AC -> CL31B475KAHNNNE; Manufacturer TDK Corporation -> Samsung Electro-Mechanics
Other:
- note added: "1206 0 ohm used in place of L1 because\nL1 is not in stock at Digi-Key as of 10/22/2020"
Changed lines of the file:
@@
 F 1 "4.7uF" H 6115 3855 50  0000 L CNN
 F 2 "Capacitor_SMD:C_1206_3216Metric_Pad1.33x1.80mm_HandSolder" H 6038 3750 50  0001 C CNN
-F 3 "https://product.tdk.com/info/en/catalog/datasheets/mlcc_commercial_general_en.pdf?ref_disty=digikey" H 6000 3900 50  0001 C CNN
-F 4 "TDK Corporation" H 6000 3900 50  0001 C CNN "Manufacturer"
-F 5 "C3216X7R1E475K160AC" H 6000 3900 50  0001 C CNN "MPN"
+F 3 "https://media.digikey.com/pdf/Data%20Sheets/Samsung%20PDFs/CL_Series_MLCC_ds.pdf" H 6000 3900 50  0001 C CNN
+F 4 "Samsung Electro-Mechanics" H 6000 3900 50  0001 C CNN "Manufacturer"
+F 5 "CL31B475KAHNNNE" H 6000 3900 50  0001 C CNN "MPN"
 	1    6000 3900
 	1    0    0    -1
@@
 	5150 3750 5050 3750
 Connection ~ 5050 3750
-Text Notes 4450 3500 0    50   ~ 0
+Text Notes 3600 3800 0    50   ~ 0
 V_in Range: 4.5-18 V
 Text HLabel 6750 3950 0    50   Input ~ 0
@@
 Wire Wire Line
 	6500 3750 6800 3750
+Text Notes 4650 3250 0    50   ~ 0
+1206 0 ohm used in place of L1 because\nL1 is not in stock at Digi-Key as of 10/22/2020
 $EndSCHEMATC
