File: KiCad Files/DC-DC Converter.sch (KiCad schematic (older format))
At the start: 4 parts, among them U2 TEC2-1219WI

Commit message: Updated part numbers to match
Updated part numbers on components to fix errors.
Parts:
- U2: MPN (none) -> TEC2-1219WI; Manufacturer (none) -> TRACO Power
Changed lines of the file:
@@
 F 2 "Converter_DCDC:Converter_DCDC_TRACO_TMR-xxxx_THT" H 7300 3600 50  0001 C CNN
 F 3 "https://www.tracopower.com/products/tec2wi.pdf" H 7300 3450 50  0001 C CNN
+F 4 "TEC2-1219WI" H 7300 3950 50  0001 C CNN "MPN"
+F 5 "TRACO Power" H 7300 3950 50  0001 C CNN "Manufacturer"
 	1    7300 3950
 	1    0    0    -1
