File: KiCad Files/Programmer Board.sch (KiCad schematic (older format))
At the start: 13 parts, among them J10 Conn_01x03, J2 Conn_01x03, J7 302-S101, J9 Conn_02x18_Odd_Even

Commit message: Updated part numbers to match
Updated part numbers on components to fix errors.
Parts:
- E2: MPN 105-1103-001 -> 575-4
- E4: Digi-Key_PN J577-ND -> 36-575-4-ND; MPN 36-575-4-ND -> 575-4
Changed lines of the file:
@@
 F 3 "http://keyelco.com/userAssets/file/M65p111.pdf" H 3050 3100 60  0001 L CNN
 F 4 "36-575-4-ND" H 3050 3200 60  0001 L CNN "Digi-Key_PN"
-F 5 "105-1103-001" H 3050 3300 60  0001 L CNN "MPN"
+F 5 "575-4" H 3050 3300 60  0001 L CNN "MPN"
 F 6 "Connectors, Interconnects" H 3050 3400 60  0001 L CNN "Category"
 F 7 "Banana and Tip Connectors - Jacks, Plugs" H 3050 3500 60  0001 L CNN "Family"
@@
 F 2 "LMS-6_Interface_Board:575_Banana_Jack" H 7750 1900 60  0001 L CNN
 F 3 "http://keyelco.com/userAssets/file/M65p111.pdf" H 7750 2000 60  0001 L CNN
-F 4 "J577-ND" H 7750 2100 60  0001 L CNN "Digi-Key_PN"
-F 5 "36-575-4-ND" H 7750 2200 60  0001 L CNN "MPN"
+F 4 "36-575-4-ND" H 7750 2100 60  0001 L CNN "Digi-Key_PN"
+F 5 "575-4" H 7750 2200 60  0001 L CNN "MPN"
 F 6 "Connectors, Interconnects" H 7750 2300 60  0001 L CNN "Category"
 F 7 "Banana and Tip Connectors - Jacks, Plugs" H 7750 2400 60  0001 L CNN "Family"
